File: hardware/h43it_micro/h43bit_micro.kicad_sch (KiCad schematic)
At the start: 25 parts, among them J1 Conn_01x04_Pin, SW1 SW_Push, U1 ATtiny414-SS

Commit message: first draft of schematic
Parts:
- J1: footprint (none) -> Connector_PinHeader_2.54mm:PinHeader_1x04_P2.54mm_Vertical
- SW1: footprint (none) -> MyLib:PTS526 SM15 SMTR2 LFS
Changed lines of the file:
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@@
       (effects (font (size 1.27 1.27)))
     )
-    (property "Footprint" "" (at 88.9 43.18 0)
+    (property "Footprint" "Connector_PinHeader_2.54mm:PinHeader_1x04_P2.54mm_Vertical" (at 88.9 43.18 0)
       (effects (font (size 1.27 1.27)) hide)
     )
@@
       (effects (font (size 1.27 1.27)))
     )
-    (property "Footprint" "" (at 123.19 39.37 0)
-      (effects (font (size 1.27 1.27)) hide)
-    )
+    (property "Footprint" "MyLib:PTS526 SM15 SMTR2 LFS" (at 123.19 39.37 0)
+      (effects (font (size 1.27 1.27)) hide)
+    )

Commit message: circular tracks
Parts:
- BT1: footprint (none) -> MyLib:BAT-HLD-001
- C1: footprint (none) -> Capacitor_SMD:C_0805_2012Metric
- D1, D10, D11, D12, D13, D14, D15, D16, D2, D3, D4, D5, D6, D7, D8, D9: footprint (none) -> LED_SMD:LED_0805_2012Metric
- R1, R2, R3, R4: footprint (none) -> Resistor_SMD:R_0805_2012Metric
Connections:
- net L- is gone; now on net M-: U1.11 (PA1)
- net M-: no longer U1.12 (PA2)
- net N-: now also U1.12 (PA2); no longer U1.13 (PA3)
- net O-: now also U1.13 (PA3); no longer U1.2 (PA4)
- net P-: now also U1.2 (PA4)
Changed lines of the file:
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@@
+    (stroke (width 0) (type default))
+  )
+  (wire (pts (xy 83.82 110.49) (xy 83.82 116.84))
     (stroke (width 0) (type default))
   )
@@
     (stroke (width 0) (type default))
   )
-  (wire (pts (xy 83.82 110.49) (xy 83.82 116.84))
-    (stroke (width 0) (type default))
-  )
   (wire (pts (xy 48.26 166.37) (xy 52.07 166.37))
     (stroke (width 0) (type default))
@@
     (effects (font (size 1.27 1.27)) (justify left bottom))
   )
-  (label "M-" (at 102.87 87.63 0) (fields_autoplaced)
-    (effects (font (size 1.27 1.27)) (justify left bottom))
-  )
-  (label "O-" (at 102.87 92.71 0) (fields_autoplaced)
+  (label "N-" (at 102.87 87.63 0) (fields_autoplaced)
+    (effects (font (size 1.27 1.27)) (justify left bottom))
+  )
+  (label "P-" (at 102.87 92.71 0) (fields_autoplaced)
     (effects (font (size 1.27 1.27)) (justify left bottom))
   )
@@
     (effects (font (size 1.27 1.27)) (justify left bottom))
   )
-  (label "L-" (at 102.87 85.09 0) (fields_autoplaced)
+  (label "M-" (at 102.87 85.09 0) (fields_autoplaced)
     (effects (font (size 1.27 1.27)) (justify left bottom))
   )
@@
     (effects (font (size 1.27 1.27)) (justify left bottom))
   )
-  (label "N-" (at 102.87 90.17 0) (fields_autoplaced)
+  (label "O-" (at 102.87 90.17 0) (fields_autoplaced)
     (effects (font (size 1.27 1.27)) (justify left bottom))
   )
@@
       (effects (font (size 1.27 1.27)))
     )
-    (property "Footprint" "" (at 66.294 159.004 90)
+    (property "Footprint" "Resistor_SMD:R_0805_2012Metric" (at 66.294 159.004 90)
       (effects (font (size 1.27 1.27)) hide)
     )
@@
       (effects (font (size 1.27 1.27)))
     )
-    (property "Footprint" "" (at 107.95 179.07 0)
+    (property "Footprint" "LED_SMD:LED_0805_2012Metric" (at 107.95 179.07 0)
       (effects (font (size 1.27 1.27)) hide)
     )
@@
       (effects (font (size 1.27 1.27)))
     )
-    (property "Footprint" "" (at 139.7 179.07 0)
+    (property "Footprint" "LED_SMD:LED_0805_2012Metric" (at 139.7 179.07 0)
       (effects (font (size 1.27 1.27)) hide)
     )
@@
       (effects (font (size 1.27 1.27)) (justify left))
     )
-    (property "Footprint" "" (at 26.3652 48.26 0)
+    (property "Footprint" "Capacitor_SMD:C_0805_2012Metric" (at 26.3652 48.26 0)
       (effects (font (size 1.27 1.27)) hide)
     )
@@
       (effects (font (size 1.27 1.27)))
     )
-    (property "Footprint" "" (at 139.7 140.97 0)
+    (property "Footprint" "LED_SMD:LED_0805_2012Metric" (at 139.7 140.97 0)
       (effects (font (size 1.27 1.27)) hide)
     )
@@
       (effects (font (size 1.27 1.27)))
     )
-    (property "Footprint" "" (at 76.2 140.97 0)
+    (property "Footprint" "LED_SMD:LED_0805_2012Metric" (at 76.2 140.97 0)
       (effects (font (size 1.27 1.27)) hide)
     )
@@
       (effects (font (size 1.27 1.27)))
     )
-    (property "Footprint" "" (at 44.45 140.97 0)
+    (property "Footprint" "LED_SMD:LED_0805_2012Metric" (at 44.45 140.97 0)
       (effects (font (size 1.27 1.27)) hide)
     )
@@
       (effects (font (size 1.27 1.27)))
     )
-    (property "Footprint" "" (at 76.2 179.07 0)
+    (property "Footprint" "LED_SMD:LED_0805_2012Metric" (at 76.2 179.07 0)
       (effects (font (size 1.27 1.27)) hide)
     )
@@
       (effects (font (size 1.27 1.27)))
     )
-    (property "Footprint" "" (at 107.95 153.67 0)
+    (property "Footprint" "LED_SMD:LED_0805_2012Metric" (at 107.95 153.67 0)
       (effects (font (size 1.27 1.27)) hide)
     )
@@
       (effects (font (size 1.27 1.27)))
     )
-    (property "Footprint" "" (at 107.95 140.97 0)
+    (property "Footprint" "LED_SMD:LED_0805_2012Metric" (at 107.95 140.97 0)
       (effects (font (size 1.27 1.27)) hide)
     )
@@
       (effects (font (size 1.27 1.27)))
     )
-    (property "Footprint" "" (at 76.2 153.67 0)
+    (property "Footprint" "LED_SMD:LED_0805_2012Metric" (at 76.2 153.67 0)
       (effects (font (size 1.27 1.27)) hide)
     )
@@
       (effects (font (size 1.27 1.27)))
     )
-    (property "Footprint" "" (at 107.95 166.37 0)
+    (property "Footprint" "LED_SMD:LED_0805_2012Metric" (at 107.95 166.37 0)
       (effects (font (size 1.27 1.27)) hide)
     )
@@
       (effects (font (size 1.27 1.27)))
     )
-    (property "Footprint" "" (at 34.544 159.004 90)
+    (property "Footprint" "Resistor_SMD:R_0805_2012Metric" (at 34.544 159.004 90)
       (effects (font (size 1.27 1.27)) hide)
     )
@@
       (effects (font (size 1.27 1.27)))
     )
-    (property "Footprint" "" (at 44.45 153.67 0)
+    (property "Footprint" "LED_SMD:LED_0805_2012Metric" (at 44.45 153.67 0)
       (effects (font (size 1.27 1.27)) hide)
     )
@@
       (effects (font (size 1.27 1.27)))
     )
-    (property "Footprint" "" (at 76.2 166.37 0)
+    (property "Footprint" "LED_SMD:LED_0805_2012Metric" (at 76.2 166.37 0)
       (effects (font (size 1.27 1.27)) hide)
     )
@@
       (effects (font (size 1.27 1.27)))
     )
-    (property "Footprint" "" (at 139.7 166.37 0)
+    (property "Footprint" "LED_SMD:LED_0805_2012Metric" (at 139.7 166.37 0)
       (effects (font (size 1.27 1.27)) hide)
     )
@@
       (effects (font (size 1.27 1.27)) (justify left))
     )
-    (property "Footprint" "" (at 40.64 44.196 90)
+    (property "Footprint" "MyLib:BAT-HLD-001" (at 40.64 44.196 90)
       (effects (font (size 1.27 1.27)) hide)
     )
@@
       (effects (font (size 1.27 1.27)))
     )
-    (property "Footprint" "" (at 98.044 159.004 90)
+    (property "Footprint" "Resistor_SMD:R_0805_2012Metric" (at 98.044 159.004 90)
       (effects (font (size 1.27 1.27)) hide)
     )
@@
       (effects (font (size 1.27 1.27)))
     )
-    (property "Footprint" "" (at 129.794 159.004 90)
+    (property "Footprint" "Resistor_SMD:R_0805_2012Metric" (at 129.794 159.004 90)
       (effects (font (size 1.27 1.27)) hide)
     )
@@
       (effects (font (size 1.27 1.27)))
     )
-    (property "Footprint" "" (at 139.7 153.67 0)
+    (property "Footprint" "LED_SMD:LED_0805_2012Metric" (at 139.7 153.67 0)
       (effects (font (size 1.27 1.27)) hide)
     )
@@
       (effects (font (size 1.27 1.27)))
     )
-    (property "Footprint" "" (at 44.45 179.07 0)
+    (property "Footprint" "LED_SMD:LED_0805_2012Metric" (at 44.45 179.07 0)
       (effects (font (size 1.27 1.27)) hide)
     )
@@
       (effects (font (size 1.27 1.27)))
     )
-    (property "Footprint" "" (at 44.45 166.37 0)
-      (effects (font (size 1.27 1.27)) hide)
-    )
+    (property "Footprint" "LED_SMD:LED_0805_2012Metric" (at 44.45 166.37 0)
+      (effects (font (size 1.27 1.27)) hide)
+    )

Commit message: first draft of a finished pcb
Parts:
- added SW2: SW_Push, MyLib:FSM2JSMAATR, symbol Switch:SW_Push
Connections:
- net C+: now also U1.4 (PA6); no longer U1.6 (PB3)
- net D+: now also U1.3 (PA5); no longer U1.4 (PA6)
- net GND: now also SW2.1
- net SW: now also SW2.2

Commit message: switch SW on micro
Connections:
- net C+: now also U1.5 (PA7); no longer U1.4 (PA6)
- net SW: now also U1.4 (PA6); no longer U1.5 (PA7)
Changed lines of the file:
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@@
     (stroke (width 0) (type default))
   )
-  (wire (pts (xy 105.41 100.33) (xy 99.06 100.33))
+  (wire (pts (xy 102.87 97.79) (xy 99.06 97.79))
     (stroke (width 0) (type default))
   )
@@
     (stroke (width 0) (type default))
   )
+  (wire (pts (xy 102.87 100.33) (xy 99.06 100.33))
+    (stroke (width 0) (type default))
+  )
   (wire (pts (xy 64.77 82.55) (xy 68.58 82.55))
     (stroke (width 0) (type default))
@@
     (stroke (width 0) (type default))
   )
-  (wire (pts (xy 99.06 97.79) (xy 102.87 97.79))
-    (stroke (width 0) (type default))
-  )
   (wire (pts (xy 80.01 140.97) (xy 83.82 140.97))
     (stroke (width 0) (type default))
@@
     (effects (font (size 1.27 1.27)) (justify left bottom))
   )
-  (label "C+" (at 102.87 97.79 0) (fields_autoplaced)
+  (label "C+" (at 102.87 100.33 0) (fields_autoplaced)
     (effects (font (size 1.27 1.27)) (justify left bottom))
   )
@@
     (effects (font (size 1.27 1.27)) (justify left bottom))
   )
-  (label "SW" (at 105.41 100.33 0) (fields_autoplaced)
-    (effects (font (size 1.27 1.27)) (justify left bottom))
-  )
+  (label "SW" (at 102.87 97.79 0) (fields_autoplaced)
+    (effects (font (size 1.27 1.27)) (justify left bottom))
+  )
