File: hardware/h43it_micro/h43bit_micro.kicad_pcb (KiCad board)
At the start: 2 copper layers, 41 x 41 mm, 26 parts, among them J1 Conn_01x04_Pin, SW1 SW_Push, SW2 SW_Push, U1 ATtiny414-SS

Commit message: recreate production files
Parts:
- moved J1 1.02 mm to (112.5, 94.7)
Routing:
- net /SW: track 29.8 -> 28.8 mm
Changed lines of the file:
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@@
   )
   (footprint "Connector_PinHeader_2.54mm:PinHeader_1x04_P2.54mm_Vertical" (layer "F.Cu")
-    (at 111.506 94.742)
+    (at 112.522 94.742)
     (descr "Through hole straight pin header, 1x04, 2.54mm pitch, single row")
     (tags "Through hole pin header THT 1x04 2.54mm single row")
@@
   (segment (start 96.796 107.138) (end 96.818 107.116) (width 0.25) (layer "F.Cu") (net 2))
   (segment (start 97.017001 99.939) (end 94.488 102.468001) (width 0.25) (layer "F.Cu") (net 2))
-  (segment (start 97.642001 98.044) (end 98.617 98.044) (width 0.25) (layer "F.Cu") (net 2))
   (segment (start 96.796 108.676) (end 96.796 107.138) (width 0.25) (layer "F.Cu") (net 2))
   (segment (start 98.552 93.886439) (end 98.617 93.951439) (width 0.25) (layer "F.Cu") (net 4))
@@
   (segment (start 91.409224 112.746952) (end 88.986 115.170176) (width 0.25) (layer "F.Cu") (net 16))
   (arc (start 99.75 118.999999) (mid 89.205771 115.638001) (end 82.323285 106.971099) (width 0.25) (layer "F.Cu") (net 16))
-  (segment (start 91.092932 86.692372) (end 90.807628 86.692372) (width 0.25) (layer "F.Cu") (net 17))
-  (segment (start 90.807628 86.692372) (end 90.75 86.75) (width 0.25) (layer "F.Cu") (net 17))
   (segment (start 89.004718 84.604158) (end 89.004718 84.504718) (width 0.25) (layer "F.Cu") (net 17))
   (segment (start 91.092932 86.692372) (end 89.004718 84.604158) (width 0.25) (layer "F.Cu") (net 17))

Commit message: success all DRC
Parts:
- moved J1 0.68 mm to (112.1, 94.2)
Routing:
- net /TX: track 30.8 -> 14.5 mm, vias 2 -> 0
- net /A+: track 29.3 -> 20.3 mm
- net /M-: track 75.4 -> 81.0 mm
- net /UPDI: track 9.20 -> 14.5 mm
- net /B+: track 10.5 -> 11.7 mm
- net VCC: track 43.9 -> 44.6 mm
