File: hardware/h43it_macro/h43it_macro.kicad_pcb (KiCad board)
At the start: 2 copper layers, 90 x 90 mm, 48 parts, among them J1 Conn_01x04_Pin, SW2 SW_Push, U4 ATtiny816-S

Commit message: pcb for macro 4
Parts:
- moved C3 11.8 mm to (125.5, 90.1), turned to -90 degrees
- moved U2 7.06 mm to (134.6, 90.3)
- moved C2 5.36 mm to (129.2, 90.3), turned to -90 degrees
Routing:
- net GND: track 20.1 -> 0.00 mm, vias 2 -> 0
- net /CapSens-IO1: track 29.8 -> 18.0 mm, vias 2 -> 1
- net /CapSens-IO2: track 10.9 -> 0.00 mm
- net Net-(U2-VREG): track 18.0 -> 7.98 mm, vias 2 -> 0
- net Net-(U2-CX): track 28.5 -> 25.5 mm
Changed lines of the file:
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@@
   )
   (footprint "Capacitor_SMD:C_0805_2012Metric" (layer "F.Cu")
-    (at 132.5 99.5)
+    (at 125.48 90.066 -90)
     (descr "Capacitor SMD 0805 (2012 Metric), square (rectangular) end terminal, IPC_7351 nominal, (Body size source: IPC-SM-782 page 76, https://www.pcb-3d.com/wordpress/wp-content/uploads/ipc-sm-782a_amendment_1_and_2.pdf, https://docs.google.com/spreadsheets/d/1BsfQQcO9C6DZCsRaXUlFlo91Tg2WpOkGARC1WS5S8t0/edit?usp=sharing), generated with kicad-footprint-generator")
     (tags "capacitor")
@@
     (property "ki_keywords" "cap capacitor")
     (attr smd)
-    (fp_text reference "C3" (at 0 -1.68) (layer "F.SilkS")
-        (effects (font (size 1 1) (thickness 0.15)))
-    )
-    (fp_text value "1uF" (at 0 1.68) (layer "F.Fab")
-        (effects (font (size 1 1) (thickness 0.15)))
-    )
-    (fp_text user "${REFERENCE}" (at 0 0) (layer "F.Fab")
+    (fp_text reference "C3" (at 0 -1.68 90) (layer "F.SilkS")
+        (effects (font (size 1 1) (thickness 0.15)))
+    )
+    (fp_text value "1uF" (at 0 1.68 90) (layer "F.Fab")
+        (effects (font (size 1 1) (thickness 0.15)))
+    )
+    (fp_text user "${REFERENCE}" (at 0 0 90) (layer "F.Fab")
         (effects (font (size 0.5 0.5) (thickness 0.08)))
     )
@@
     (fp_line (start 1 0.625) (end -1 0.625)
       (stroke (width 0.1) (type solid)) (layer "F.Fab"))
-    (pad "1" smd roundrect (at -0.95 0) (size 1 1.45) (layers "F.Cu" "F.Paste" "F.Mask") (roundrect_rratio 0.25)
+    (pad "1" smd roundrect (at -0.95 0 270) (size 1 1.45) (layers "F.Cu" "F.Paste" "F.Mask") (roundrect_rratio 0.25)
       (net 26 "Net-(U2-VREG)") (pintype "passive"))
-    (pad "2" smd roundrect (at 0.95 0) (size 1 1.45) (layers "F.Cu" "F.Paste" "F.Mask") (roundrect_rratio 0.25)
+    (pad "2" smd roundrect (at 0.95 0 270) (size 1 1.45) (layers "F.Cu" "F.Paste" "F.Mask") (roundrect_rratio 0.25)
       (net 2 "GND") (pintype "passive"))
     (model "${KICAD6_3DMODEL_DIR}/Capacitor_SMD.3dshapes/C_0805_2012Metric.wrl"
@@
   )
   (footprint "Capacitor_SMD:C_0805_2012Metric" (layer "F.Cu")
-    (at 132.5 94.5)
+    (at 129.224 90.254 -90)
     (descr "Capacitor SMD 0805 (2012 Metric), square (rectangular) end terminal, IPC_7351 nominal, (Body size source: IPC-SM-782 page 76, https://www.pcb-3d.com/wordpress/wp-content/uploads/ipc-sm-782a_amendment_1_and_2.pdf, https://docs.google.com/spreadsheets/d/1BsfQQcO9C6DZCsRaXUlFlo91Tg2WpOkGARC1WS5S8t0/edit?usp=sharing), generated with kicad-footprint-generator")
     (tags "capacitor")
@@
     (property "ki_keywords" "cap capacitor")
     (attr smd)
-    (fp_text reference "C2" (at 0 -1.68) (layer "F.SilkS")
-        (effects (font (size 1 1) (thickness 0.15)))
-    )
-    (fp_text value "100pF" (at 0 1.68) (layer "F.Fab")
-        (effects (font (size 1 1) (thickness 0.15)))
-    )
-    (fp_text user "${REFERENCE}" (at 0 0) (layer "F.Fab")
+    (fp_text reference "C2" (at 0 -1.68 90) (layer "F.SilkS")
+        (effects (font (size 1 1) (thickness 0.15)))
+    )
+    (fp_text value "100pF" (at 0 1.68 90) (layer "F.Fab")
+        (effects (font (size 1 1) (thickness 0.15)))
+    )
+    (fp_text user "${REFERENCE}" (at 0 0 90) (layer "F.Fab")
         (effects (font (size 0.5 0.5) (thickness 0.08)))
     )
@@
     (fp_line (start 1 0.625) (end -1 0.625)
       (stroke (width 0.1) (type solid)) (layer "F.Fab"))
-    (pad "1" smd roundrect (at -0.95 0) (size 1 1.45) (layers "F.Cu" "F.Paste" "F.Mask") (roundrect_rratio 0.25)
+    (pad "1" smd roundrect (at -0.95 0 270) (size 1 1.45) (layers "F.Cu" "F.Paste" "F.Mask") (roundrect_rratio 0.25)
       (net 26 "Net-(U2-VREG)") (pintype "passive"))
-    (pad "2" smd roundrect (at 0.95 0) (size 1 1.45) (layers "F.Cu" "F.Paste" "F.Mask") (roundrect_rratio 0.25)
+    (pad "2" smd roundrect (at 0.95 0 270) (size 1 1.45) (layers "F.Cu" "F.Paste" "F.Mask") (roundrect_rratio 0.25)
       (net 2 "GND") (pintype "passive"))
     (model "${KICAD6_3DMODEL_DIR}/Capacitor_SMD.3dshapes/C_0805_2012Metric.wrl"
@@
   )
   (footprint "MyLib:TSOT32-6" (layer "F.Cu")
-    (at 127.5 90.5 90)
+    (at 134.558 90.32 90)
     (property "Sheetfile" "h43it_macro.kicad_sch")
     (property "Sheetname" "")
@@
   (segment (start 99.5 88.5) (end 94.5 88.5) (width 0.25) (layer "F.Cu") (net 1))
   (segment (start 110.35 87.15) (end 110.35 88.415) (width 0.25) (layer "F.Cu") (net 1))
-  (segment (start 128.7 90.5) (end 127.52 90.5) (width 0.25) (layer "F.Cu") (net 2))
-  (segment (start 117.667 88.415) (end 117.54 88.542) (width 0.25) (layer "F.Cu") (net 2))
-  (segment (start 119.65 88.415) (end 117.667 88.415) (width 0.25) (layer "F.Cu") (net 2))
-  (segment (start 127.52 90.5) (end 127.446 90.574) (width 0.25) (layer "F.Cu") (net 2))
-  (via (at 127.446 90.574) (size 0.8) (drill 0.4) (layers "F.Cu" "B.Cu") (net 2))
-  (via (at 117.54 88.542) (size 0.8) (drill 0.4) (layers "F.Cu" "B.Cu") (net 2))
-  (segment (start 126.300305 95.225) (end 124.223 95.225) (width 0.25) (layer "B.Cu") (net 2))
-  (segment (start 127.446 94.079305) (end 126.300305 95.225) (width 0.25) (layer "B.Cu") (net 2))
-  (segment (start 127.446 90.574) (end 127.446 94.079305) (width 0.25) (layer "B.Cu") (net 2))
-  (segment (start 124.223 95.225) (end 117.54 88.542) (width 0.25) (layer "B.Cu") (net 2))
   (segment (start 111.5 109.9565) (end 111.5 107.995) (width 0.25) (layer "F.Cu") (net 3))
   (segment (start 80 29.9375) (end 85 34.9375) (width 0.25) (layer "F.Cu") (net 3))
@@
   (segment (start 122.366 86.275) (end 122.366 90.32) (width 0.25) (layer "B.Cu") (net 23))
   (segment (start 108.015 89.685) (end 107.888 89.558) (width 0.25) (layer "F.Cu") (net 24))
-  (segment (start 128.7 91.45) (end 129.35 91.45) (width 0.25) (layer "F.Cu") (net 24))
-  (segment (start 129.35 91.45) (end 129.425 91.375) (width 0.25) (layer "F.Cu") (net 24))
-  (segment (start 128.208 87.526) (end 121.803 87.526) (width 0.25) (layer "F.Cu") (net 24))
-  (segment (start 129.425 88.743) (end 128.208 87.526) (width 0.25) (layer "F.Cu") (net 24))
-  (segment (start 129.425 91.375) (end 129.425 88.743) (width 0.25) (layer "F.Cu") (net 24))
   (segment (start 111.374999 89.685) (end 110.35 89.685) (width 0.25) (layer "F.Cu") (net 24))
   (segment (start 110.35 89.685) (end 108.015 89.685) (width 0.25) (layer "F.Cu") (net 24))
-  (segment (start 121.803 87.526) (end 121.604 87.725) (width 0.25) (layer "F.Cu") (net 24))
   (via (at 107.888 89.558) (size 0.8) (drill 0.4) (layers "F.Cu" "B.Cu") (net 24))
-  (via (at 121.604 87.725) (size 0.8) (drill 0.4) (layers "F.Cu" "B.Cu") (net 24))
   (segment (start 121.604 87.725) (end 109.721 87.725) (width 0.25) (layer "B.Cu") (net 24))
   (segment (start 109.721 87.725) (end 107.888 89.558) (width 0.25) (layer "B.Cu") (net 24))
-  (segment (start 128.7 88.7) (end 128 88) (width 0.25) (layer "F.Cu") (net 25))
-  (segment (start 128 88) (end 123.5 88) (width 0.25) (layer "F.Cu") (net 25))
-  (segment (start 121.815 89.685) (end 119.65 89.685) (width 0.25) (layer "F.Cu") (net 25))
-  (segment (start 123.5 88) (end 121.815 89.685) (width 0.25) (layer "F.Cu") (net 25))
-  (segment (start 128.7 89.55) (end 128.7 88.7) (width 0.25) (layer "F.Cu") (net 25))
-  (segment (start 131.55 94.5) (end 126 94.5) (width 0.25) (layer "F.Cu") (net 26))
-  (segment (start 124.55 89.55) (end 124.5 89.5) (width 0.25) (layer "F.Cu") (net 26))
-  (segment (start 131.55 94.5) (end 131.55 99.5) (width 0.25) (layer "F.Cu") (net 26))
-  (segment (start 126.3 89.55) (end 124.55 89.55) (width 0.25) (layer "F.Cu") (net 26))
-  (via (at 124.5 89.5) (size 0.8) (drill 0.4) (layers "F.Cu" "B.Cu") (net 26))
-  (via (at 126 94.5) (size 0.8) (drill 0.4) (layers "F.Cu" "B.Cu") (net 26))
-  (segment (start 124.5 89.5) (end 124.5 93) (width 0.25) (layer "B.Cu") (net 26))
-  (segment (start 124.5 93) (end 126 94.5) (width 0.25) (layer "B.Cu") (net 26))
-  (segment (start 123.275 91.45) (end 126.3 91.45) (width 0.25) (layer "F.Cu") (net 28))
+  (segment (start 129.29 89.37) (end 129.224 89.304) (width 0.25) (layer "F.Cu") (net 26))
+  (segment (start 133.358 89.37) (end 129.29 89.37) (width 0.25) (layer "F.Cu") (net 26))
+  (segment (start 125.668 89.304) (end 125.48 89.116) (width 0.25) (layer "F.Cu") (net 26))
+  (segment (start 129.224 89.304) (end 125.668 89.304) (width 0.25) (layer "F.Cu") (net 26))
   (segment (start 123.225 91.5) (end 123.2 91.475) (width 0.25) (layer "F.Cu") (net 28))
   (segment (start 123.225 91.5) (end 123.275 91.45) (width 0.25) (layer "F.Cu") (net 28))

Commit message: tiny changes and added R6
Parts:
- added CapSens-IO1: SolderJumper_2_Bridged, Jumper:SolderJumper-2_P1.3mm_Bridged_RoundedPad1.0x1.5mm, B.Cu at (115.0, 93.7)
- added CapSens_IO2: SolderJumper_2_Open, Jumper:SolderJumper-2_P1.3mm_Open_RoundedPad1.0x1.5mm, B.Cu at (115.0, 90.1)
- added R6: 42R, Resistor_SMD:R_0805_2012Metric, F.Cu at (129.7, 94.2)
- added SWITCH1: SolderJumper_2_Open, Jumper:SolderJumper-2_P1.3mm_Open_RoundedPad1.0x1.5mm, B.Cu at (115.0, 97.2)
- moved C1 4.90 mm to (99.4, 89.5)
- moved C4 4.70 mm to (104.2, 89.4)
- moved C2 0.51 mm to (129.7, 90.3)
- moved C3 0.48 mm to (125.9, 90.3)
- moved U2 0.33 mm to (134.5, 90.0)
Connections:
- U4 pad 18: /SW -> /interrupt_pin
- U4 pad 19: /CapSens-IO2 -> /SW
Routing:
- net /CapSens-IO1: track 18.0 -> 46.0 mm, vias 1 -> 3
- net /CapSens-IO2: track 0.00 -> 21.2 mm, vias 0 -> 1
- net Net-(U2-CX): track 25.5 -> 40.9 mm
- net /interrupt_pin: track 0.00 -> 15.0 mm, vias 0 -> 1
- net /SW: track 19.4 -> 28.1 mm, vias 2 -> 3
- net Net-(U2-VDDHI): track 0.00 -> 6.16 mm
- net VCC: track 88.0 -> 83.0 mm

Commit message: no errors in macro
Parts:
- moved R2 0.44 mm to (152.4, 61.5)
- moved R4 0.43 mm to (78.6, 58.5)
- moved R1 0.42 mm to (115.0, 34.1)
- moved R3 0.27 mm to (116.5, 106.7)
Routing:
- net /P-: track 320.0 -> 326.2 mm, vias 3 -> 4
- net /CapSens-IO1: track 46.0 -> 47.8 mm
- net VCC: track 83.0 -> 81.1 mm
- net /A+: track 112.6 -> 113.4 mm
- net /B+: track 61.0 -> 61.7 mm
